Commit message: Enabling use with other packages

File: khi_description/urdf/cx/khi.ros2_control.xacro (robot description, xacro)
@@ -56,4 +56,6 @@
         <param name="type"> ${jt1_type} </param>
         <param name="arm">arm1</param>
+        <param name="initial_position">0.0</param>
+        <param name="initial_velocity">0.0</param>
       </joint>
       <joint name="${prefix}joint2">
@@ -67,4 +69,6 @@
         <param name="type"> ${jt2_type} </param>
         <param name="arm">arm1</param>
+        <param name="initial_position">0.0</param>
+        <param name="initial_velocity">0.0</param>
       </joint>
       <joint name="${prefix}joint3">
@@ -78,4 +82,6 @@
         <param name="type"> ${jt3_type} </param>
         <param name="arm">arm1</param>
+        <param name="initial_position">0.0</param>
+        <param name="initial_velocity">0.0</param>
       </joint>
       <joint name="${prefix}joint4">
@@ -89,4 +95,6 @@
         <param name="type"> ${jt4_type} </param>
         <param name="arm">arm1</param>
+        <param name="initial_position">0.0</param>
+        <param name="initial_velocity">0.0</param>
       </joint>
       <joint name="${prefix}joint5">
@@ -100,4 +108,6 @@
         <param name="type"> ${jt5_type} </param>
         <param name="arm">arm1</param>
+        <param name="initial_position">0.0</param>
+        <param name="initial_velocity">0.0</param>
       </joint>
       <joint name="${prefix}joint6">
@@ -111,4 +121,6 @@
         <param name="type"> ${jt6_type} </param>
         <param name="arm">arm1</param>
+        <param name="initial_position">0.0</param>
+        <param name="initial_velocity">0.0</param>
       </joint>
       <xacro:if value="${use_gazebo}">

File: khi_description/urdf/cx/khi_joint_link.xacro (robot description, xacro)
@@ -5,12 +5,12 @@
     <xacro:include filename="$(find khi_description)/urdf/$(arg robot_series)/get_joint_limits.xacro"/>
     <xacro:include filename="$(find khi_description)/urdf/material.xacro"/>
-    <!-- Fix robot to world -->
-    <link name="world"/>
-    <!-- Joint  -->
+    <!-- Fix robot to world
+    <link name="world"/>-->
+    <!-- Joint
     <joint name="${prefix}world2base" type="fixed">
       <parent link="world"/>
       <child link="${prefix}base_link"/>
       <origin xyz="0 0 0" rpy="0 0 0" />
-    </joint>
+    </joint>-->
     <joint name="${prefix}joint1" type="${jt1_type}">
       <axis xyz="${axis1}" />
