Commit message: fixed ros2_control node naming bug

File: khi_description/urdf/cx/khi.ros2_control.xacro (robot description, xacro)
@@ -20,5 +20,6 @@
     ft_sensor
     ">
-    <ros2_control name="${robot_name}" type="system">
+    <xacro:property name="safe_robot_name" value="${robot_name.replace('-', '_')}" />
+    <ros2_control name="${safe_robot_name}" type="system">
       <xacro:include filename="$(find khi_description)/urdf/$(arg robot_series)/get_mechanical_parameters.xacro"/>
       <xacro:include filename="$(find khi_description)/urdf/$(arg robot_series)/get_joint_limits.xacro"/>
