Commit message: Corrected naming of mesh files for CX robots

File: khi_description/urdf/cx/khi_joint_link.xacro (robot description, xacro)
@@ -70,5 +70,5 @@
             <mesh filename="package://khi_description/meshes/${robot_series}/${robot_name}/J0.dae"/>
           </xacro:if>
-          <mesh filename="package://khi_description/meshes/${robot_series}/${robot_name}/J0.stl"/>
+          <mesh filename="package://khi_description/meshes/${robot_series}/${robot_name}/J0.dae"/>
         </geometry>
         <xacro:white/>
@@ -80,5 +80,5 @@
             <mesh filename="package://khi_description/meshes/${robot_series}/${robot_name}/J0.dae"/>
           </xacro:if>
-          <mesh filename="package://khi_description/meshes/${robot_series}/${robot_name}/J0.stl"/>
+          <mesh filename="package://khi_description/meshes/${robot_series}/${robot_name}/J0.dae"/>
         </geometry>
         <xacro:white/>
@@ -97,5 +97,5 @@
             <mesh filename="package://khi_description/meshes/${robot_series}/${robot_name}/J1.dae"/>
           </xacro:if>
-          <mesh filename="package://khi_description/meshes/${robot_series}/${robot_name}/J1.stl"/>
+          <mesh filename="package://khi_description/meshes/${robot_series}/${robot_name}/J1.dae"/>
         </geometry>
         <xacro:white/>
@@ -107,5 +107,5 @@
             <mesh filename="package://khi_description/meshes/${robot_series}/${robot_name}/J1.dae"/>
           </xacro:if>
-          <mesh filename="package://khi_description/meshes/${robot_series}/${robot_name}/J1.stl"/>
+          <mesh filename="package://khi_description/meshes/${robot_series}/${robot_name}/J1.dae"/>
         </geometry>
         <origin xyz="0 0 0" rpy="${radians(l1_rpy_x)} ${radians(l1_rpy_y)} ${radians(l1_rpy_z)}"/>
@@ -123,5 +123,5 @@
             <mesh filename="package://khi_description/meshes/${robot_series}/${robot_name}/J2.dae"/>
           </xacro:if>
-          <mesh filename="package://khi_description/meshes/${robot_series}/${robot_name}/J2.stl"/>
+          <mesh filename="package://khi_description/meshes/${robot_series}/${robot_name}/J2.dae"/>
         </geometry>
         <xacro:white/>
@@ -133,5 +133,5 @@
             <mesh filename="package://khi_description/meshes/${robot_series}/${robot_name}/J2.dae"/>
           </xacro:if>
-          <mesh filename="package://khi_description/meshes/${robot_series}/${robot_name}/J2.stl"/>
+          <mesh filename="package://khi_description/meshes/${robot_series}/${robot_name}/J2.dae"/>
         </geometry>
         <origin xyz="0 0 0" rpy="${radians(l2_rpy_x)} ${radians(l2_rpy_y)} ${radians(l2_rpy_z)}"/>
@@ -149,5 +149,5 @@
             <mesh filename="package://khi_description/meshes/${robot_series}/${robot_name}/J3.dae"/>
           </xacro:if>
-          <mesh filename="package://khi_description/meshes/${robot_series}/${robot_name}/J3.stl"/>
+          <mesh filename="package://khi_description/meshes/${robot_series}/${robot_name}/J3.dae"/>
         </geometry>
         <xacro:white/>
@@ -159,5 +159,5 @@
             <mesh filename="package://khi_description/meshes/${robot_series}/${robot_name}/J3.dae"/>
           </xacro:if>
-          <mesh filename="package://khi_description/meshes/${robot_series}/${robot_name}/J3.stl"/>
+          <mesh filename="package://khi_description/meshes/${robot_series}/${robot_name}/J3.dae"/>
         </geometry>
         <origin xyz="0 0 0" rpy="${radians(l3_rpy_x)} ${radians(l3_rpy_y)} ${radians(l3_rpy_z)}"/>
@@ -175,5 +175,5 @@
             <mesh filename="package://khi_description/meshes/${robot_series}/${robot_name}/J4.dae"/>
           </xacro:if>
-          <mesh filename="package://khi_description/meshes/${robot_series}/${robot_name}/J4.stl"/>
+          <mesh filename="package://khi_description/meshes/${robot_series}/${robot_name}/J4.dae"/>
         </geometry>
         <xacro:white/>
@@ -185,5 +185,5 @@
             <mesh filename="package://khi_description/meshes/${robot_series}/${robot_name}/J4.dae"/>
           </xacro:if>
-          <mesh filename="package://khi_description/meshes/${robot_series}/${robot_name}/J4.stl"/>
+          <mesh filename="package://khi_description/meshes/${robot_series}/${robot_name}/J4.dae"/>
         </geometry>
         <origin xyz="${l4_x} ${l4_y} ${l4_z}" rpy="${radians(l4_rpy_x)} ${radians(l4_rpy_y)} ${radians(l4_rpy_z)}"/>
@@ -201,5 +201,5 @@
             <mesh filename="package://khi_description/meshes/${robot_series}/${robot_name}/J5.dae"/>
           </xacro:if>
-          <mesh filename="package://khi_description/meshes/${robot_series}/${robot_name}/J5.stl"/>
+          <mesh filename="package://khi_description/meshes/${robot_series}/${robot_name}/J5.dae"/>
         </geometry>
         <xacro:white/>
@@ -211,5 +211,5 @@
             <mesh filename="package://khi_description/meshes/${robot_series}/${robot_name}/J5.dae"/>
           </xacro:if>
-          <mesh filename="package://khi_description/meshes/${robot_series}/${robot_name}/J5.stl"/>
+          <mesh filename="package://khi_description/meshes/${robot_series}/${robot_name}/J5.dae"/>
         </geometry>
         <origin xyz="0 0 0" rpy="${radians(l5_rpy_x)} ${radians(l5_rpy_y)} ${radians(l5_rpy_z)}"/>
@@ -227,5 +227,5 @@
             <mesh filename="package://khi_description/meshes/${robot_series}/${robot_name}/J6.dae"/>
           </xacro:if>
-          <mesh filename="package://khi_description/meshes/${robot_series}/${robot_name}/J6.stl"/>
+          <mesh filename="package://khi_description/meshes/${robot_series}/${robot_name}/J6.dae"/>
         </geometry>
         <xacro:white/>
@@ -237,5 +237,5 @@
             <mesh filename="package://khi_description/meshes/${robot_series}/${robot_name}/J6.dae"/>
           </xacro:if>
-          <mesh filename="package://khi_description/meshes/${robot_series}/${robot_name}/J6.stl"/>
+          <mesh filename="package://khi_description/meshes/${robot_series}/${robot_name}/J6.dae"/>
         </geometry>
         <origin xyz="0 0 0" rpy="${radians(l6_rpy_x)} ${radians(l6_rpy_y)} ${radians(l6_rpy_z)}"/>

Commit message: Added more moveit changes

File: khi_description/urdf/cx/khi_joint_link.xacro (robot description, xacro)
@@ -68,7 +68,8 @@
       <visual>
         <geometry>
-          <xacro:if value="${robot_name=='cx110l-bc01' or robot_name=='cx165l-bc01'}">
+          <xacro:if value="${robot_name=='cx110l-bc01' or robot_name=='cx165l_bc01'}">
             <mesh filename="package://khi_description/meshes/${robot_series}/${robot_name}/J0.stl"/>
           </xacro:if>
+          <mesh filename="package://khi_description/meshes/${robot_series}/${robot_name}/J0.stl"/>
         </geometry>
         <xacro:white/>
@@ -77,7 +78,8 @@
       <collision>
         <geometry>
-          <xacro:if value="${robot_name=='cx110l-bc01' or robot_name=='cx165l-bc01'}">
+          <xacro:if value="${robot_name=='cx110l-bc01' or robot_name=='cx165l_bc01'}">
             <mesh filename="package://khi_description/meshes/${robot_series}/${robot_name}/J0.stl"/>
           </xacro:if>
+          <mesh filename="package://khi_description/meshes/${robot_series}/${robot_name}/J0.stl"/>
         </geometry>
         <xacro:white/>
@@ -93,7 +95,8 @@
       <visual>
         <geometry>
-          <xacro:if value="${robot_name=='cx110l-bc01' or robot_name=='cx165l-bc01'}">
+          <xacro:if value="${robot_name=='cx110l-bc01' or robot_name=='cx165l_bc01'}">
             <mesh filename="package://khi_description/meshes/${robot_series}/${robot_name}/J1.stl"/>
           </xacro:if>
+          <mesh filename="package://khi_description/meshes/${robot_series}/${robot_name}/J1.stl"/>
         </geometry>
         <xacro:white/>
@@ -102,7 +105,8 @@
       <collision>
         <geometry>
-          <xacro:if value="${robot_name=='cx110l-bc01' or robot_name=='cx165l-bc01'}">
+          <xacro:if value="${robot_name=='cx110l-bc01' or robot_name=='cx165l_bc01'}">
             <mesh filename="package://khi_description/meshes/${robot_series}/${robot_name}/J1_hull.stl"/>
           </xacro:if>
+          <mesh filename="package://khi_description/meshes/${robot_series}/${robot_name}/J1_hull.stl"/>
         </geometry>
         <origin xyz="0 0 0" rpy="${radians(l1_rpy_x)} ${radians(l1_rpy_y)} ${radians(l1_rpy_z)}"/>
@@ -117,7 +121,8 @@
       <visual>
         <geometry>
-          <xacro:if value="${robot_name=='cx110l-bc01' or robot_name=='cx165l-bc01'}">
+          <xacro:if value="${robot_name=='cx110l-bc01' or robot_name=='cx165l_bc01'}">
             <mesh filename="package://khi_description/meshes/${robot_series}/${robot_name}/J2.stl"/>
           </xacro:if>
+          <mesh filename="package://khi_description/meshes/${robot_series}/${robot_name}/J2.stl"/>
         </geometry>
         <xacro:white/>
@@ -126,7 +131,8 @@
       <collision>
         <geometry>
-          <xacro:if value="${robot_name=='cx110l-bc01' or robot_name=='cx165l-bc01'}">
+          <xacro:if value="${robot_name=='cx110l-bc01' or robot_name=='cx165l_bc01'}">
             <mesh filename="package://khi_description/meshes/${robot_series}/${robot_name}/J2_hull.stl"/>
           </xacro:if>
+          <mesh filename="package://khi_description/meshes/${robot_series}/${robot_name}/J2_hull.stl"/>
         </geometry>
         <origin xyz="0 0 0" rpy="${radians(l2_rpy_x)} ${radians(l2_rpy_y)} ${radians(l2_rpy_z)}"/>
@@ -141,8 +147,9 @@
       <visual>
         <geometry>
-          <xacro:if value="${robot_name=='cx110l-bc01' or robot_name=='cx165l-bc01'}">
+          <xacro:if value="${robot_name=='cx110l-bc01' or robot_name=='cx165l_bc01'}">
             <mesh filename="package://khi_description/meshes/${robot_series}/${robot_name}/J3.stl"/>
           </xacro:if>
         </geometry>
+        <mesh filename="package://khi_description/meshes/${robot_series}/${robot_name}/J3.stl"/>
         <xacro:white/>
         <origin xyz="0 0 0" rpy="${radians(l3_rpy_x)} ${radians(l3_rpy_y)} ${radians(l3_rpy_z)}"/>
@@ -150,7 +157,8 @@
       <collision>
         <geometry>
-          <xacro:if value="${robot_name=='cx110l-bc01' or robot_name=='cx165l-bc01'}">
+          <xacro:if value="${robot_name=='cx110l-bc01' or robot_name=='cx165l_bc01'}">
             <mesh filename="package://khi_description/meshes/${robot_series}/${robot_name}/J3_hull.stl"/>
           </xacro:if>
+          <mesh filename="package://khi_description/meshes/${robot_series}/${robot_name}/J3_hull.stl"/>
         </geometry>
         <origin xyz="0 0 0" rpy="${radians(l3_rpy_x)} ${radians(l3_rpy_y)} ${radians(l3_rpy_z)}"/>
@@ -165,7 +173,8 @@
       <visual>
         <geometry>
-          <xacro:if value="${robot_name=='cx110l-bc01' or robot_name=='cx165l-bc01'}">
+          <xacro:if value="${robot_name=='cx110l-bc01' or robot_name=='cx165l_bc01'}">
             <mesh filename="package://khi_description/meshes/${robot_series}/${robot_name}/J4.stl"/>
           </xacro:if>
+          <mesh filename="package://khi_description/meshes/${robot_series}/${robot_name}/J4.stl"/>
         </geometry>
         <xacro:white/>
@@ -174,7 +183,8 @@
       <collision>
         <geometry>
-          <xacro:if value="${robot_name=='cx110l-bc01' or robot_name=='cx165l-bc01'}">
+          <xacro:if value="${robot_name=='cx110l-bc01' or robot_name=='cx165l_bc01'}">
             <mesh filename="package://khi_description/meshes/${robot_series}/${robot_name}/J4_hull.stl"/>
           </xacro:if>
+          <mesh filename="package://khi_description/meshes/${robot_series}/${robot_name}/J4_hull.stl"/>
         </geometry>
         <origin xyz="${l4_x} ${l4_y} ${l4_z}" rpy="${radians(l4_rpy_x)} ${radians(l4_rpy_y)} ${radians(l4_rpy_z)}"/>
@@ -189,7 +199,8 @@
       <visual>
         <geometry>
-          <xacro:if value="${robot_name=='cx110l-bc01' or robot_name=='cx165l-bc01'}">
+          <xacro:if value="${robot_name=='cx110l-bc01' or robot_name=='cx165l_bc01'}">
             <mesh filename="package://khi_description/meshes/${robot_series}/${robot_name}/J5.stl"/>
           </xacro:if>
+          <mesh filename="package://khi_description/meshes/${robot_series}/${robot_name}/J5.stl"/>
         </geometry>
         <xacro:white/>
@@ -198,7 +209,8 @@
       <collision>
         <geometry>
-          <xacro:if value="${robot_name=='cx110l-bc01' or robot_name=='cx165l-bc01'}">
+          <xacro:if value="${robot_name=='cx110l-bc01' or robot_name=='cx165l_bc01'}">
             <mesh filename="package://khi_description/meshes/${robot_series}/${robot_name}/J5_hull.stl"/>
           </xacro:if>
+          <mesh filename="package://khi_description/meshes/${robot_series}/${robot_name}/J5_hull.stl"/>
         </geometry>
         <origin xyz="0 0 0" rpy="${radians(l5_rpy_x)} ${radians(l5_rpy_y)} ${radians(l5_rpy_z)}"/>
@@ -213,7 +225,8 @@
       <visual>
         <geometry>
-          <xacro:if value="${robot_name=='cx110l-bc01' or robot_name=='cx165l-bc01'}">
+          <xacro:if value="${robot_name=='cx110l-bc01' or robot_name=='cx165l_bc01'}">
             <mesh filename="package://khi_description/meshes/${robot_series}/${robot_name}/J6.stl"/>
           </xacro:if>
+          <mesh filename="package://khi_description/meshes/${robot_series}/${robot_name}/J6.stl"/>
         </geometry>
         <xacro:white/>
@@ -222,7 +235,8 @@
       <collision>
         <geometry>
-          <xacro:if value="${robot_name=='cx110l-bc01' or robot_name=='cx165l-bc01'}">
+          <xacro:if value="${robot_name=='cx110l-bc01' or robot_name=='cx165l_bc01'}">
             <mesh filename="package://khi_description/meshes/${robot_series}/${robot_name}/J6_hull.stl"/>
           </xacro:if>
+          <mesh filename="package://khi_description/meshes/${robot_series}/${robot_name}/J6_hull.stl"/>
         </geometry>
         <origin xyz="0 0 0" rpy="${radians(l6_rpy_x)} ${radians(l6_rpy_y)} ${radians(l6_rpy_z)}"/>

Commit message: Modifications for cx165l-bc01

File: khi_description/urdf/cx/khi_joint_link.xacro (robot description, xacro)
@@ -68,7 +68,7 @@
         <geometry>
           <xacro:if value="${robot_name=='cx110l-bc01'}">
-            <mesh filename="package://khi_description/meshes/${robot_series}/${robot_name}/J0.dae"/>
-          </xacro:if>
-          <mesh filename="package://khi_description/meshes/${robot_series}/${robot_name}/J0.dae"/>
+            <mesh filename="package://khi_description/meshes/${robot_series}/${robot_name}/J0.stl"/>
+          </xacro:if>
+          <mesh filename="package://khi_description/meshes/${robot_series}/${robot_name}/J0.stl"/>
         </geometry>
         <xacro:white/>
@@ -78,7 +78,7 @@
         <geometry>
           <xacro:if value="${robot_name=='cx110l-bc01'}">
-            <mesh filename="package://khi_description/meshes/${robot_series}/${robot_name}/J0.dae"/>
-          </xacro:if>
-          <mesh filename="package://khi_description/meshes/${robot_series}/${robot_name}/J0.dae"/>
+            <mesh filename="package://khi_description/meshes/${robot_series}/${robot_name}/J0.stl"/>
+          </xacro:if>
+          <mesh filename="package://khi_description/meshes/${robot_series}/${robot_name}/J0.stl"/>
         </geometry>
         <xacro:white/>
@@ -95,7 +95,7 @@
         <geometry>
           <xacro:if value="${robot_name=='cx110l-bc01'}">
-            <mesh filename="package://khi_description/meshes/${robot_series}/${robot_name}/J1.dae"/>
-          </xacro:if>
-          <mesh filename="package://khi_description/meshes/${robot_series}/${robot_name}/J1.dae"/>
+            <mesh filename="package://khi_description/meshes/${robot_series}/${robot_name}/J1.stl"/>
+          </xacro:if>
+          <mesh filename="package://khi_description/meshes/${robot_series}/${robot_name}/J1.stl"/>
         </geometry>
         <xacro:white/>
@@ -105,7 +105,7 @@
         <geometry>
           <xacro:if value="${robot_name=='cx110l-bc01'}">
-            <mesh filename="package://khi_description/meshes/${robot_series}/${robot_name}/J1.dae"/>
-          </xacro:if>
-          <mesh filename="package://khi_description/meshes/${robot_series}/${robot_name}/J1.dae"/>
+            <mesh filename="package://khi_description/meshes/${robot_series}/${robot_name}/J1.stl"/>
+          </xacro:if>
+          <mesh filename="package://khi_description/meshes/${robot_series}/${robot_name}/J1.stl"/>
         </geometry>
         <origin xyz="0 0 0" rpy="${radians(l1_rpy_x)} ${radians(l1_rpy_y)} ${radians(l1_rpy_z)}"/>
@@ -121,7 +121,7 @@
         <geometry>
           <xacro:if value="${robot_name=='cx110l-bc01'}">
-            <mesh filename="package://khi_description/meshes/${robot_series}/${robot_name}/J2.dae"/>
-          </xacro:if>
-          <mesh filename="package://khi_description/meshes/${robot_series}/${robot_name}/J2.dae"/>
+            <mesh filename="package://khi_description/meshes/${robot_series}/${robot_name}/J2.stl"/>
+          </xacro:if>
+          <mesh filename="package://khi_description/meshes/${robot_series}/${robot_name}/J2.stl"/>
         </geometry>
         <xacro:white/>
@@ -131,7 +131,7 @@
         <geometry>
           <xacro:if value="${robot_name=='cx110l-bc01'}">
-            <mesh filename="package://khi_description/meshes/${robot_series}/${robot_name}/J2.dae"/>
-          </xacro:if>
-          <mesh filename="package://khi_description/meshes/${robot_series}/${robot_name}/J2.dae"/>
+            <mesh filename="package://khi_description/meshes/${robot_series}/${robot_name}/J2.stl"/>
+          </xacro:if>
+          <mesh filename="package://khi_description/meshes/${robot_series}/${robot_name}/J2.stl"/>
         </geometry>
         <origin xyz="0 0 0" rpy="${radians(l2_rpy_x)} ${radians(l2_rpy_y)} ${radians(l2_rpy_z)}"/>
@@ -147,7 +147,7 @@
         <geometry>
           <xacro:if value="${robot_name=='cx110l-bc01'}">
-            <mesh filename="package://khi_description/meshes/${robot_series}/${robot_name}/J3.dae"/>
-          </xacro:if>
-          <mesh filename="package://khi_description/meshes/${robot_series}/${robot_name}/J3.dae"/>
+            <mesh filename="package://khi_description/meshes/${robot_series}/${robot_name}/J3.stl"/>
+          </xacro:if>
+          <mesh filename="package://khi_description/meshes/${robot_series}/${robot_name}/J3.stl"/>
         </geometry>
         <xacro:white/>
@@ -157,7 +157,7 @@
         <geometry>
           <xacro:if value="${robot_name=='cx110l-bc01'}">
-            <mesh filename="package://khi_description/meshes/${robot_series}/${robot_name}/J3.dae"/>
-          </xacro:if>
-          <mesh filename="package://khi_description/meshes/${robot_series}/${robot_name}/J3.dae"/>
+            <mesh filename="package://khi_description/meshes/${robot_series}/${robot_name}/J3.stl"/>
+          </xacro:if>
+          <mesh filename="package://khi_description/meshes/${robot_series}/${robot_name}/J3.stl"/>
         </geometry>
         <origin xyz="0 0 0" rpy="${radians(l3_rpy_x)} ${radians(l3_rpy_y)} ${radians(l3_rpy_z)}"/>
@@ -173,7 +173,7 @@
         <geometry>
           <xacro:if value="${robot_name=='cx110l-bc01'}">
-            <mesh filename="package://khi_description/meshes/${robot_series}/${robot_name}/J4.dae"/>
-          </xacro:if>
-          <mesh filename="package://khi_description/meshes/${robot_series}/${robot_name}/J4.dae"/>
+            <mesh filename="package://khi_description/meshes/${robot_series}/${robot_name}/J4.stl"/>
+          </xacro:if>
+          <mesh filename="package://khi_description/meshes/${robot_series}/${robot_name}/J4.stl"/>
         </geometry>
         <xacro:white/>
@@ -183,7 +183,7 @@
         <geometry>
           <xacro:if value="${robot_name=='cx110l-bc01'}">
-            <mesh filename="package://khi_description/meshes/${robot_series}/${robot_name}/J4.dae"/>
-          </xacro:if>
-          <mesh filename="package://khi_description/meshes/${robot_series}/${robot_name}/J4.dae"/>
+            <mesh filename="package://khi_description/meshes/${robot_series}/${robot_name}/J4.stl"/>
+          </xacro:if>
+          <mesh filename="package://khi_description/meshes/${robot_series}/${robot_name}/J4.stl"/>
         </geometry>
         <origin xyz="${l4_x} ${l4_y} ${l4_z}" rpy="${radians(l4_rpy_x)} ${radians(l4_rpy_y)} ${radians(l4_rpy_z)}"/>
@@ -199,7 +199,7 @@
         <geometry>
           <xacro:if value="${robot_name=='cx110l-bc01'}">
-            <mesh filename="package://khi_description/meshes/${robot_series}/${robot_name}/J5.dae"/>
-          </xacro:if>
-          <mesh filename="package://khi_description/meshes/${robot_series}/${robot_name}/J5.dae"/>
+            <mesh filename="package://khi_description/meshes/${robot_series}/${robot_name}/J5.stl"/>
+          </xacro:if>
+          <mesh filename="package://khi_description/meshes/${robot_series}/${robot_name}/J5.stl"/>
         </geometry>
         <xacro:white/>
@@ -209,7 +209,7 @@
         <geometry>
           <xacro:if value="${robot_name=='cx110l-bc01'}">
-            <mesh filename="package://khi_description/meshes/${robot_series}/${robot_name}/J5.dae"/>
-          </xacro:if>
-          <mesh filename="package://khi_description/meshes/${robot_series}/${robot_name}/J5.dae"/>
+            <mesh filename="package://khi_description/meshes/${robot_series}/${robot_name}/J5.stl"/>
+          </xacro:if>
+          <mesh filename="package://khi_description/meshes/${robot_series}/${robot_name}/J5.stl"/>
         </geometry>
         <origin xyz="0 0 0" rpy="${radians(l5_rpy_x)} ${radians(l5_rpy_y)} ${radians(l5_rpy_z)}"/>
@@ -225,7 +225,7 @@
         <geometry>
           <xacro:if value="${robot_name=='cx110l-bc01'}">
-            <mesh filename="package://khi_description/meshes/${robot_series}/${robot_name}/J6.dae"/>
-          </xacro:if>
-          <mesh filename="package://khi_description/meshes/${robot_series}/${robot_name}/J6.dae"/>
+            <mesh filename="package://khi_description/meshes/${robot_series}/${robot_name}/J6.stl"/>
+          </xacro:if>
+          <mesh filename="package://khi_description/meshes/${robot_series}/${robot_name}/J6.stl"/>
         </geometry>
         <xacro:white/>
@@ -235,7 +235,7 @@
         <geometry>
           <xacro:if value="${robot_name=='cx110l-bc01'}">
-            <mesh filename="package://khi_description/meshes/${robot_series}/${robot_name}/J6.dae"/>
-          </xacro:if>
-          <mesh filename="package://khi_description/meshes/${robot_series}/${robot_name}/J6.dae"/>
+            <mesh filename="package://khi_description/meshes/${robot_series}/${robot_name}/J6.stl"/>
+          </xacro:if>
+          <mesh filename="package://khi_description/meshes/${robot_series}/${robot_name}/J6.stl"/>
         </geometry>
         <origin xyz="0 0 0" rpy="${radians(l6_rpy_x)} ${radians(l6_rpy_y)} ${radians(l6_rpy_z)}"/>
