Commit message: Added proper moveit config and fixed meshes.

File: khi_description/srdf/cx/khi_macro.srdf.xacro (robot description, xacro)
@@ -29,4 +29,6 @@
     <!--END EFFECTOR: Purpose: Represent information about an end effector.-->
     <end_effector name="${prefix}moveit_ee" parent_link="${prefix}link6" group="${prefix}tool" parent_group="${prefix}manipulator" />
+    <!--Groups kinematic plugins -->
+    <kinematics_plugin_config filename="package://khi_moveit/config/kinematics.yaml"/>
     <!--DISABLE COLLISIONS: By default it is assumed that any link of the robot could potentially come into collision with any other link in the robot. This tag disables collision checking between a specified pair of links. -->
     <disable_collisions link1="${prefix}base_link" link2="${prefix}link1" reason="Adjacent" />

File: khi_description/urdf/cx/khi_joint_link.xacro (robot description, xacro)
@@ -64,11 +64,11 @@
     </joint>
     <!-- Link  -->
+    <!-- Link  -->
     <link name="${prefix}base_link">
       <visual>
         <geometry>
-          <xacro:if value="${robot_name=='cx110l-bc01'}">
-            <mesh filename="package://khi_description/meshes/${robot_series}/${robot_name}/J0.dae"/>
-          </xacro:if>
-          <mesh filename="package://khi_description/meshes/${robot_series}/${robot_name}/J0.dae"/>
+          <xacro:if value="${robot_name=='cx110l-bc01' or robot_name=='cx165l-bc01'}">
+            <mesh filename="package://khi_description/meshes/${robot_series}/${robot_name}/J0.stl"/>
+          </xacro:if>
         </geometry>
         <xacro:white/>
@@ -77,8 +77,7 @@
       <collision>
         <geometry>
-          <xacro:if value="${robot_name=='cx110l-bc01'}">
-            <mesh filename="package://khi_description/meshes/${robot_series}/${robot_name}/J0.dae"/>
-          </xacro:if>
-          <mesh filename="package://khi_description/meshes/${robot_series}/${robot_name}/J0.dae"/>
+          <xacro:if value="${robot_name=='cx110l-bc01' or robot_name=='cx165l-bc01'}">
+            <mesh filename="package://khi_description/meshes/${robot_series}/${robot_name}/J0.stl"/>
+          </xacro:if>
         </geometry>
         <xacro:white/>
@@ -94,8 +93,7 @@
       <visual>
         <geometry>
-          <xacro:if value="${robot_name=='cx110l-bc01'}">
-            <mesh filename="package://khi_description/meshes/${robot_series}/${robot_name}/J1.dae"/>
-          </xacro:if>
-          <mesh filename="package://khi_description/meshes/${robot_series}/${robot_name}/J1.dae"/>
+          <xacro:if value="${robot_name=='cx110l-bc01' or robot_name=='cx165l-bc01'}">
+            <mesh filename="package://khi_description/meshes/${robot_series}/${robot_name}/J1.stl"/>
+          </xacro:if>
         </geometry>
         <xacro:white/>
@@ -104,8 +102,7 @@
       <collision>
         <geometry>
-          <xacro:if value="${robot_name=='cx110l-bc01'}">
-            <mesh filename="package://khi_description/meshes/${robot_series}/${robot_name}/J1.dae"/>
-          </xacro:if>
-          <mesh filename="package://khi_description/meshes/${robot_series}/${robot_name}/J1.dae"/>
+          <xacro:if value="${robot_name=='cx110l-bc01' or robot_name=='cx165l-bc01'}">
+            <mesh filename="package://khi_description/meshes/${robot_series}/${robot_name}/J1_hull.stl"/>
+          </xacro:if>
         </geometry>
         <origin xyz="0 0 0" rpy="${radians(l1_rpy_x)} ${radians(l1_rpy_y)} ${radians(l1_rpy_z)}"/>
@@ -120,8 +117,7 @@
       <visual>
         <geometry>
-          <xacro:if value="${robot_name=='cx110l-bc01'}">
-            <mesh filename="package://khi_description/meshes/${robot_series}/${robot_name}/J2.dae"/>
-          </xacro:if>
-          <mesh filename="package://khi_description/meshes/${robot_series}/${robot_name}/J2.dae"/>
+          <xacro:if value="${robot_name=='cx110l-bc01' or robot_name=='cx165l-bc01'}">
+            <mesh filename="package://khi_description/meshes/${robot_series}/${robot_name}/J2.stl"/>
+          </xacro:if>
         </geometry>
         <xacro:white/>
@@ -130,8 +126,7 @@
       <collision>
         <geometry>
-          <xacro:if value="${robot_name=='cx110l-bc01'}">
-            <mesh filename="package://khi_description/meshes/${robot_series}/${robot_name}/J2.dae"/>
-          </xacro:if>
-          <mesh filename="package://khi_description/meshes/${robot_series}/${robot_name}/J2.dae"/>
+          <xacro:if value="${robot_name=='cx110l-bc01' or robot_name=='cx165l-bc01'}">
+            <mesh filename="package://khi_description/meshes/${robot_series}/${robot_name}/J2_hull.stl"/>
+          </xacro:if>
         </geometry>
         <origin xyz="0 0 0" rpy="${radians(l2_rpy_x)} ${radians(l2_rpy_y)} ${radians(l2_rpy_z)}"/>
@@ -146,8 +141,7 @@
       <visual>
         <geometry>
-          <xacro:if value="${robot_name=='cx110l-bc01'}">
-            <mesh filename="package://khi_description/meshes/${robot_series}/${robot_name}/J3.dae"/>
-          </xacro:if>
-          <mesh filename="package://khi_description/meshes/${robot_series}/${robot_name}/J3.dae"/>
+          <xacro:if value="${robot_name=='cx110l-bc01' or robot_name=='cx165l-bc01'}">
+            <mesh filename="package://khi_description/meshes/${robot_series}/${robot_name}/J3.stl"/>
+          </xacro:if>
         </geometry>
         <xacro:white/>
@@ -156,8 +150,7 @@
       <collision>
         <geometry>
-          <xacro:if value="${robot_name=='cx110l-bc01'}">
-            <mesh filename="package://khi_description/meshes/${robot_series}/${robot_name}/J3.dae"/>
-          </xacro:if>
-          <mesh filename="package://khi_description/meshes/${robot_series}/${robot_name}/J3.dae"/>
+          <xacro:if value="${robot_name=='cx110l-bc01' or robot_name=='cx165l-bc01'}">
+            <mesh filename="package://khi_description/meshes/${robot_series}/${robot_name}/J3_hull.stl"/>
+          </xacro:if>
         </geometry>
         <origin xyz="0 0 0" rpy="${radians(l3_rpy_x)} ${radians(l3_rpy_y)} ${radians(l3_rpy_z)}"/>
@@ -172,8 +165,7 @@
       <visual>
         <geometry>
-          <xacro:if value="${robot_name=='cx110l-bc01'}">
-            <mesh filename="package://khi_description/meshes/${robot_series}/${robot_name}/J4.dae"/>
-          </xacro:if>
-          <mesh filename="package://khi_description/meshes/${robot_series}/${robot_name}/J4.dae"/>
+          <xacro:if value="${robot_name=='cx110l-bc01' or robot_name=='cx165l-bc01'}">
+            <mesh filename="package://khi_description/meshes/${robot_series}/${robot_name}/J4.stl"/>
+          </xacro:if>
         </geometry>
         <xacro:white/>
@@ -182,8 +174,7 @@
       <collision>
         <geometry>
-          <xacro:if value="${robot_name=='cx110l-bc01'}">
-            <mesh filename="package://khi_description/meshes/${robot_series}/${robot_name}/J4.dae"/>
-          </xacro:if>
-          <mesh filename="package://khi_description/meshes/${robot_series}/${robot_name}/J4.dae"/>
+          <xacro:if value="${robot_name=='cx110l-bc01' or robot_name=='cx165l-bc01'}">
+            <mesh filename="package://khi_description/meshes/${robot_series}/${robot_name}/J4_hull.stl"/>
+          </xacro:if>
         </geometry>
         <origin xyz="${l4_x} ${l4_y} ${l4_z}" rpy="${radians(l4_rpy_x)} ${radians(l4_rpy_y)} ${radians(l4_rpy_z)}"/>
@@ -198,8 +189,7 @@
       <visual>
         <geometry>
-          <xacro:if value="${robot_name=='cx110l-bc01'}">
-            <mesh filename="package://khi_description/meshes/${robot_series}/${robot_name}/J5.dae"/>
-          </xacro:if>
-          <mesh filename="package://khi_description/meshes/${robot_series}/${robot_name}/J5.dae"/>
+          <xacro:if value="${robot_name=='cx110l-bc01' or robot_name=='cx165l-bc01'}">
+            <mesh filename="package://khi_description/meshes/${robot_series}/${robot_name}/J5.stl"/>
+          </xacro:if>
         </geometry>
         <xacro:white/>
@@ -208,8 +198,7 @@
       <collision>
         <geometry>
-          <xacro:if value="${robot_name=='cx110l-bc01'}">
-            <mesh filename="package://khi_description/meshes/${robot_series}/${robot_name}/J5.dae"/>
-          </xacro:if>
-          <mesh filename="package://khi_description/meshes/${robot_series}/${robot_name}/J5.dae"/>
+          <xacro:if value="${robot_name=='cx110l-bc01' or robot_name=='cx165l-bc01'}">
+            <mesh filename="package://khi_description/meshes/${robot_series}/${robot_name}/J5_hull.stl"/>
+          </xacro:if>
         </geometry>
         <origin xyz="0 0 0" rpy="${radians(l5_rpy_x)} ${radians(l5_rpy_y)} ${radians(l5_rpy_z)}"/>
@@ -224,8 +213,7 @@
       <visual>
         <geometry>
-          <xacro:if value="${robot_name=='cx110l-bc01'}">
-            <mesh filename="package://khi_description/meshes/${robot_series}/${robot_name}/J6.dae"/>
-          </xacro:if>
-          <mesh filename="package://khi_description/meshes/${robot_series}/${robot_name}/J6.dae"/>
+          <xacro:if value="${robot_name=='cx110l-bc01' or robot_name=='cx165l-bc01'}">
+            <mesh filename="package://khi_description/meshes/${robot_series}/${robot_name}/J6.stl"/>
+          </xacro:if>
         </geometry>
         <xacro:white/>
@@ -234,8 +222,7 @@
       <collision>
         <geometry>
-          <xacro:if value="${robot_name=='cx110l-bc01'}">
-            <mesh filename="package://khi_description/meshes/${robot_series}/${robot_name}/J6.dae"/>
-          </xacro:if>
-          <mesh filename="package://khi_description/meshes/${robot_series}/${robot_name}/J6.dae"/>
+          <xacro:if value="${robot_name=='cx110l-bc01' or robot_name=='cx165l-bc01'}">
+            <mesh filename="package://khi_description/meshes/${robot_series}/${robot_name}/J6_hull.stl"/>
+          </xacro:if>
         </geometry>
         <origin xyz="0 0 0" rpy="${radians(l6_rpy_x)} ${radians(l6_rpy_y)} ${radians(l6_rpy_z)}"/>
